Commit message: oil bottle urdf

File: urdf/oil_bottle.urdf (robot description, URDF)
Before this commit: robot oil_bottle, 1 links, 0 joints
Links:
- link bottle: geometry collision mesh filename=oil_bottle_big.stl scale=0.0254 0.0254 0.0254; visual mesh filename=oil_bottle_big.stl scale=0.0254 0.0254 0.0254
