Commit message: Across-the-board updates to get optotrak frames agreeing with kinect, and so on

File: urdf/irb140_chull_ati_gelsight.urdf (robot description, URDF)
Before this commit: robot IRB140_ATI_GELSIGHT, 9 links, 8 joints
Links:
- added link ati_endplate; visual cylinder length=.01 radius=0.04
Joints:
- added joint ati_endplate_joint: type fixed, parent link_6, child ati_endplate, origin xyz=0.05 0 0 rpy=3.1415 -1.579 0.0
- joint gelsight_box_joint: origin xyz=0.098 0 0 rpy=3.1415 -1.579 0.0 -> xyz=0.105 0 0 rpy=3.1415 -1.579 0.0

Commit message: Lots of tweaks to improve operation for demo for russ RSS '16.

File: urdf/irb140_chull_ati_gelsight.urdf (robot description, URDF)
Before this commit: robot IRB140_ATI_GELSIGHT, 10 links, 9 joints
Links:
- link gelsight_box: geometry collision box size=0.033 0.033 0.031; visual box size=0.033 0.033 0.031
Joints:
- joint gelsight_box_joint: origin xyz=0.105 0 0 rpy=3.1415 -1.579 0.0 -> xyz=0.09814 0 0 rpy=3.1415 -1.579 0.0

File: urdf/irb140_chull_ati_gelsight_no_collision.urdf (robot description, URDF)
Before this commit: robot IRB140_ATI_GELSIGHT, 10 links, 9 joints
Links:
- link gelsight_box: geometry visual box size=0.033 0.033 0.031
Joints:
- joint gelsight_box_joint: origin xyz=0.105 0 0 rpy=3.1415 -1.579 0.0 -> xyz=0.09814 0 0 rpy=3.1415 -1.579 0.0
