Commit message: Working demonstration of IRB140+Gelsight testsetup Things that work: - Separate manipulationTracker configs for groundtruth, transform-generation, and tracking with gelsight+kinect - Apriltag fitting util for director Things that don't work: - Collision geometry for gelsight box is nonexistent, we need collision groups in drake for this to work properly - Tracking is absymal - Covariance estimates are not well founded - No optitrak, groundtruth tracking still has errors on order of cm

File: urdf/desk.urdf (robot description, URDF)
Before this commit: robot desk, 1 links, 0 joints
Links:
- link desk: geometry collision box size=0.32 0.45 0.04; visual box size=0.32 0.45 0.04

Commit message: Modifications across board to try to get this producing good data. Sunlight is wrecking my ground truth now

File: urdf/desk.urdf (robot description, URDF)
Before this commit: robot desk, 1 links, 0 joints
Links:
- link desk: geometry collision box size=0.8 0.8 0.04; visual box size=0.8 0.8 0.04

File: urdf/irb140_chull_ati_gelsight_no_collision.urdf (robot description, URDF)
Before this commit: robot IRB140_ATI_GELSIGHT, 10 links, 9 joints
Links:
- link ati_endplate: geometry visual cylinder length=.01 radius=0.04
- link gelsight_box: geometry visual box size=0.033 0.033 0.033

Commit message: Replicated box pushing experiment well enough

File: urdf/desk.urdf (robot description, URDF)
Before this commit: robot desk, 1 links, 0 joints
Links:
- link desk: geometry collision box size=0.45 0.45 0.04; visual box size=0.45 0.45 0.04
