Commit message: PUBLISHED STATE. Estimtr params/code for publish
This was the state of the estimator code at the
time that we took the data that we submitted to
ICRA2017

File: urdf/hole_box.urdf (robot description, URDF)
Before this commit: robot hole_box, 1 links, 0 joints
Links:
- link hole_box: geometry collision box size=0.154 0.101 0.051; visual box size=0.154 0.101 0.051
