Commit message: Gelsight sim and tinybolt demo

File: urdf/tiny_bolt.urdf (robot description, URDF)
Before this commit: robot bolt, 2 links, 1 joints
Links:
- link body: geometry collision cylinder length=.03724 radius=0.00635; visual cylinder length=.03724 radius=0.00635
- link head: geometry collision cylinder length=0.01285 radius=0.0095; visual cylinder length=0.01285 radius=0.0095
Joints:
- joint head_to_body: origin xyz=0 0 0.02 rpy=0 0 0 -> xyz=0 0 0.025045 rpy=0 0 0

Commit message: Nonpenetration and tinybolt tracking

File: urdf/tiny_bolt.urdf (robot description, URDF)
Before this commit: robot bolt, 2 links, 1 joints
Links:
- link body: geometry collision cylinder length=.03724 radius=0.0060; visual cylinder length=.03724 radius=0.0060

Commit message: Playing with bolt tracking

File: urdf/tiny_bolt.urdf (robot description, URDF)
Before this commit: robot bolt, 2 links, 1 joints
Links:
- removed link head
- link body: geometry collision cylinder length=.03724 radius=0.0051; visual cylinder length=.03724 radius=0.0051
Joints:
- removed joint head_to_body
